Commit message: rotation works

File: urdf/dd.urdf (robot description, URDF)
Before this commit: robot dd_model, 3 links, 2 joints
Links:
- link base_link: mass 0.5 -> 5
- link wheel1: mass 0.1 -> 1
- link wheel2: mass 0.1 -> 1
Joints:
- joint base_to_wheel1: limit effort=30 velocity=1.0 -> effort=5000 velocity=10.0
- joint base_to_wheel2: limit effort=30 velocity=1.0 -> effort=5000 velocity=10.0

Commit message: spherical support wheel added

File: urdf/dd.urdf (robot description, URDF)
Before this commit: robot dd_model, 3 links, 2 joints
Links:
- added link support, mass 1; collision sphere radius=0.1; visual sphere radius=0.1
- link base_link: geometry collision box size=1 0.2 0.1; visual box size=1 0.5 0.1
Joints:
- added joint base_to_support: type fixed, parent base_link, child support, origin xyz=-0.4 0 -0.1, axis 0 0 1
